File: printer/printer.kicad_pcb (KiCad board)
At the start: 2 copper layers, 97.8 x 62.2 mm, 29 parts

Commit message: Minor tweaks
Routing:
- net GND: track 353.7 -> 352.3 mm
- net /3V3: track 292.4 -> 293.4 mm
- net /rx: track 85.4 -> 86.0 mm
Other:
- outline, holes or cut-outs redrawn
- board text added: "G"
